Commit message: added launcher to multi, modified launchers to allow namespace launch

File: panda_description/urdf/panda.urdf.xacro (robot description, xacro)
@@ -44,4 +44,5 @@
   <!--            -->
   <!-- Prefixes -->
+  <xacro:property name="robot_name" value="$(arg name)"/>
   <xacro:property name="prefix_arm" value="$(arg prefix)"/>
   <xacro:property name="prefix_gripper" value="$(arg prefix)"/>
@@ -94,5 +95,8 @@
   <xacro:if value="$(arg ros2_control)">
     <xacro:if value="${'gz' in '$(arg ros2_control_plugin)'}">
-      <xacro:ign_ros2_control controller_parameters="$(arg ros2_controller_parameters)"/>
+      <xacro:ign_ros2_control
+        controller_parameters="$(arg ros2_controller_parameters)"
+        prefix="${robot_name}"
+      />
     </xacro:if>
   </xacro:if>
