Commit message: added multiple panda robots spawn

File: panda_description/urdf/multipanda.urdf.xacro (robot description, xacro)
@@ -37,5 +37,5 @@
   <xacro:arg name="ros2_control_command_interface" default="effort"/>
   <!-- The filepath to parameters of ROS 2 controllers -->
-  <xacro:arg name="ros2_controller_parameters" default="$(find panda_moveit_config)/config/controllers_$(arg ros2_control_command_interface).yaml"/>
+  <xacro:arg name="ros2_controller_parameters" default="$(find panda_moveit_config)/config/multi_controllers_$(arg ros2_control_command_interface).yaml"/>
   <!-- Flag to preserve fixed joints and prevent lumping when generating SDF for Gazebo -->
   <xacro:arg name="gazebo_preserve_fixed_joint" default="false"/>
@@ -47,7 +47,10 @@
   <xacro:property name="prefix_gripper" value="$(arg prefix)"/>
   <!-- Origin of arm in the world -->
+  <xacro:property name="robot_name" value="$(arg name)"/>
   <xacro:property name="world_name" value="world"/>
-  <xacro:property name="origin_xyz" value="0 0 0"/>
-  <xacro:property name="origin_rpy" value="0 0 0"/>
+  <xacro:property name="robot_1_origin_xyz" value="0.31 0 0.31"/>
+  <xacro:property name="robot_1_origin_rpy" value="0 0 0"/>
+  <xacro:property name="robot_2_origin_xyz" value="1.25 0 0.31"/>
+  <xacro:property name="robot_2_origin_rpy" value="0 0 3.1416"/>
   <!-- Offset of gripper with respect to wrist flange -->
   <xacro:property name="gripper_offset_xyz" value="0 0 0"/>
@@ -61,11 +64,45 @@
     gazebo_preserve_fixed_joint="$(arg gazebo_preserve_fixed_joint)"
   />
-  <!-- Arm -->
+  <!-- Arm1 -->
   <xacro:panda_arm
-    name="$(arg name)"
+    name="robot1_panda"
     base_parent="world"
-    prefix="${prefix_arm}"
-    origin_xyz="${origin_xyz}"
-    origin_rpy="${origin_rpy}"
+    prefix="robot1_"
+    origin_xyz="${robot_1_origin_xyz}"
+    origin_rpy="${robot_1_origin_rpy}"
+    collision="$(arg collision_arm)"
+    safety_limits="$(arg safety_limits)"
+    safety_position_margin="$(arg safety_position_margin)"
+    safety_k_position="$(arg safety_k_position)"
+    safety_k_velocity="$(arg safety_k_velocity)"
+    ros2_control="$(arg ros2_control)"
+    ros2_control_plugin="$(arg ros2_control_plugin)"
+    ros2_control_command_interface="$(arg ros2_control_command_interface)"
+    gazebo_preserve_fixed_joint="$(arg gazebo_preserve_fixed_joint)"
+    link5_color="0.2 0.8 0.3 1.0"
+  />
+  <!-- Gripper1 -->
+  <xacro:if value="$(arg gripper)">
+    <xacro:panda_gripper
+      name="robot1_panda_gripper"
+      wrist_flange="robot1_${wrist_flange_name}"
+      prefix="robot1_"
+      origin_xyz="${gripper_offset_xyz}"
+      origin_rpy="${gripper_offset_rpy}"
+      collision="$(arg collision_gripper)"
+      ros2_control="$(arg ros2_control)"
+      ros2_control_plugin="$(arg ros2_control_plugin)"
+      ros2_control_command_interface="$(arg ros2_control_command_interface)"
+      gazebo_preserve_fixed_joint="$(arg gazebo_preserve_fixed_joint)"
+      use_cam="true"
+    />
+  </xacro:if>
+    <!-- Arm2 -->
+  <xacro:panda_arm
+    name="robot2_panda"
+    base_parent="world"
+    prefix="robot2_"
+    origin_xyz="${robot_2_origin_xyz}"
+    origin_rpy="${robot_2_origin_rpy}"
     collision="$(arg collision_arm)"
     safety_limits="$(arg safety_limits)"
@@ -78,10 +115,10 @@
     gazebo_preserve_fixed_joint="$(arg gazebo_preserve_fixed_joint)"
   />
-  <!-- Gripper -->
+  <!-- Gripper2 -->
   <xacro:if value="$(arg gripper)">
     <xacro:panda_gripper
-      name="$(arg name)"
-      wrist_flange="${prefix_arm}${wrist_flange_name}"
-      prefix="${prefix_gripper}"
+      name="robot2_panda_gripper"
+      wrist_flange="robot2_${wrist_flange_name}"
+      prefix="robot2_"
       origin_xyz="${gripper_offset_xyz}"
       origin_rpy="${gripper_offset_rpy}"

File: panda_description/urdf/panda_arm.xacro (robot description, xacro)
@@ -108,4 +108,5 @@
   <xacro:property name="wrist_flange_origin_xyz" value="0 0 0.107"/>
   <xacro:property name="wrist_flange_origin_rpy" value="0 0 ${-pi/4}"/>
+  <xacro:property name="default_initial_positions_file" value="$(find panda_description)/config/initial_joint_positions.yaml"/>
   <!--       -->
   <!-- Macro -->
@@ -114,4 +115,5 @@
   <xacro:property name="default_origin_rpy" value="0 0 0"/>
   <xacro:macro name="panda_arm" params="
+    name
     base_parent
     prefix:=panda_
@@ -127,4 +129,6 @@
     ros2_control_command_interface:=effort
     gazebo_preserve_fixed_joint:=false
+    initial_positions_file:=${default_initial_positions_file}
+    link5_color:=none
   ">
     <!-- Base -->
@@ -278,4 +282,5 @@
     collision="${collision}"
     mu="${link5_mu}"
+    color="${link5_color}"
     />
     <!-- 6 -->
@@ -341,7 +346,13 @@
     gazebo_preserve_fixed_joint="${gazebo_preserve_fixed_joint}"
     />
+    <!-- name="${name}" -->
     <!-- ROS 2 control -->
     <xacro:if value="${ros2_control}">
-      <xacro:ros2_control_panda_arm prefix="${prefix}" plugin="${ros2_control_plugin}" command_interface="${ros2_control_command_interface}"/>
+      <xacro:ros2_control_panda_arm
+       name="${name}"
+       prefix="${prefix}"
+       plugin="${ros2_control_plugin}"
+       command_interface="${ros2_control_command_interface}"
+       initial_positions_file="${initial_positions_file}"/>
     </xacro:if>
   </xacro:macro>

File: panda_description/urdf/panda_gripper.xacro (robot description, xacro)
@@ -7,4 +7,5 @@
   <xacro:include filename="$(find panda_description)/urdf/panda_utils.xacro"/>
   <xacro:include filename="$(find panda_description)/urdf/panda.ros2_control"/>
+  <xacro:include filename="$(find panda_description)/urdf/sensors.xacro"/>
   <!--            -->
   <!-- Properties -->
@@ -45,4 +46,5 @@
   <xacro:property name="ee_origin_xyz" value="0 0 0.1034"/>
   <xacro:property name="ee_origin_rpy" value="0 0 0"/>
+  <xacro:property name="default_initial_positions_file" value="$(find panda_description)/config/initial_joint_positions.yaml"/>
   <!--       -->
   <!-- Macro -->
@@ -51,4 +53,5 @@
   <xacro:property name="default_origin_rpy" value="0 0 0"/>
   <xacro:macro name="panda_gripper" params="
+    name
     wrist_flange
     prefix:=panda_
@@ -60,4 +63,6 @@
     ros2_control_command_interface:=effort
     gazebo_preserve_fixed_joint:=false
+    initial_positions_file:=${default_initial_positions_file}
+    use_cam:=false
   ">
     <!-- Wrist -->
@@ -134,6 +139,25 @@
     />
     <!-- ROS 2 control -->
+    <!-- name="${name}" -->
     <xacro:if value="${ros2_control}">
-      <xacro:ros2_control_panda_gripper prefix="${prefix}" plugin="${ros2_control_plugin}" command_interface="${ros2_control_command_interface}"/>
+      <xacro:ros2_control_panda_gripper
+        name="${name}"
+        prefix="${prefix}"
+        plugin="${ros2_control_plugin}"
+        command_interface="${ros2_control_command_interface}"
+        initial_positions_file="${initial_positions_file}"/>
+    </xacro:if>
+    <!-- Camera -->
+    <!-- <xacro:property name="camera_origin_xyz" value="0.5 0 1.7"/>
+    <xacro:property name="camera_origin_rpy" value="1.5708 1.5708 0"/> -->
+    <!-- 0.47 -->
+    <xacro:property name="camera_origin_xyz" value="1.0 -0.8 1.25"/>
+    <xacro:property name="camera_origin_rpy" value="0 0.685 2.35619"/>
+    <xacro:if value="${use_cam}">
+      <xacro:camera
+        name="${prefix}gripper_camera"
+        parent="${prefix}link0"
+        joint_origin_xyz="${camera_origin_xyz}"
+        joint_origin_rpy="${camera_origin_rpy}" />
     </xacro:if>
   </xacro:macro>

File: panda_description/urdf/panda_utils.xacro (robot description, xacro)
@@ -17,4 +17,5 @@
     mesh_offset_rpy:=${mesh_offset_rpy}
     gazebo_self_collide:=false
+    color:=none
   ">
     <link name="${link_name}">
@@ -24,4 +25,9 @@
           <mesh filename="package://panda_description/meshes/visual/${mesh}.dae"/>
         </geometry>
+        <xacro:unless value="${color == 'none'}">
+          <material name="${link_name}_material">
+            <color rgba="${color}"/>
+          </material>
+        </xacro:unless>
       </visual>
       <xacro:if value="${collision}">
@@ -41,4 +47,11 @@
         <self_collide>true</self_collide>
       </xacro:if>
+      <xacro:unless value="${color == 'none'}">
+        <material>
+          <ambient>${color}</ambient>
+          <diffuse>${color}</diffuse>
+          <specular>0.1 0.1 0.1 1</specular>
+        </material>
+      </xacro:unless>
     </gazebo>
   </xacro:macro>
